File: WaterPressure.kicad_pcb (KiCad board)
At the start: 2 copper layers, 54.3 x 59.4 mm, 27 parts, among them J1 MT-30361, P1 TO220, P2 TOPUMP, P3 PSENSOR, P5 CONN_01X02, SW1 SW_PUSH, SW2 SW_PUSH, SW3 SW_PUSH, U1 S102S01, U3 74HC595

Commit message: pcb finished
Parts:
- removed P5: CONN_01X02, DG306:DG306-5.08-02
- added P4: CONN_01X02, DG306:DG306-2.54-02, F.Cu at (113.7, 92.1)
- added P6: CONN_01X02, DG306:DG306-5.08-02, F.Cu at (68.6, 94.0)
- R10, R11, R12, R13, R14, R15, R16, R17: footprint Resistors_SMD:R_0805 -> Resistors_ThroughHole:Resistor_Horizontal_RM7mm; moved to F.Cu
- R7, R8, R9: footprint Resistors_ThroughHole:Resistor_Vertical_RM5mm -> Resistors_ThroughHole:Resistor_Horizontal_RM7mm
- moved R7 114.3 mm to (28.6, 130.8)
- moved R8 104.3 mm to (30.5, 128.3)
- moved P3 93.3 mm to (68.6, 109.2), turned to 270 degrees
- moved SW2 88.2 mm to (63.5, 141.0)
- moved SW3 84.0 mm to (55.2, 131.4)
- moved U1 83.5 mm to (108.0, 90.8), turned to 180 degrees
- moved R3 82.2 mm to (105.4, 97.2), turned to 270 degrees
- moved P1 73.6 mm to (92.7, 97.8)
- moved D2 64.8 mm to (111.1, 99.7)
- moved SW1 62.4 mm to (65.4, 131.4)
- moved R9 62.1 mm to (64.8, 125.1)
- moved R5 55.4 mm to (30.5, 125.7), turned to 180 degrees
- moved P2 53.5 mm to (81.3, 97.8)
- moved D1 52.6 mm to (28.6, 120.7), turned to 270 degrees
- moved R4 52.1 mm to (27.3, 118.7), turned to 0 degrees
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Connections:
- D2 pad 2: PINPUMP -> Net-(D2-Pad2)
- P2 pad 1: Net-(P1-Pad2) -> Net-(P2-Pad1)
- P2 pad 2: Net-(P2-Pad2) -> Net-(P1-Pad1)
- P3 pad 2: +5V -> GND
- P3 pad 3: GND -> +5V
- SHIELD1 pad 10: DISCLOCK -> BTN1
- SHIELD1 pad 11: DISLATCH -> LEDG
- SHIELD1 pad 12: DISDATA -> LEDR
- SHIELD1 pad 13: PINPUMP -> (no net)
- SHIELD1 pad 2: BTN1 -> DISDIGI3
- SHIELD1 pad 3: BTN2 -> DISDIGI2
- SHIELD1 pad 4: BTN3 -> DISDIGI1
- SHIELD1 pad 5: LEDG -> DISDATA
- SHIELD1 pad 5V: (no net) -> +5V
- SHIELD1 pad 6: LEDR -> DISLATCH
- SHIELD1 pad 7: DISDIGI3 -> DISCLOCK
- SHIELD1 pad 8: DISDIGI2 -> BTN3
- SHIELD1 pad 9: DISDIGI1 -> BTN2
- SHIELD1 pad AD1: (no net) -> PINPUMP
- SHIELD1 pad GND1: (no net) -> GND
- SHIELD1 pad GND2: (no net) -> GND
- SHIELD1 pad GND3: (no net) -> GND
- U1 pad 1: Net-(P1-Pad1) -> Net-(P1-Pad2)
- U1 pad 2: Net-(P2-Pad2) -> Net-(P2-Pad1)
- U1 pad 4: GND -> Net-(P4-Pad1)
Routing:
- net (no net): track 655.4 -> 0.00 mm
- net GND: track 172.7 -> 113.6 mm
- net Net-(R12-Pad2): track 62.7 -> 4.86 mm
- net Net-(J1-Pad11): track 0.00 -> 57.8 mm
- net BTN2: track 96.6 -> 45.5 mm
- net Net-(P2-Pad1): track 0.00 -> 42.5 mm
- net Net-(R13-Pad2): track 46.0 -> 4.86 mm
- net Net-(J1-Pad10): track 2.23 -> 35.6 mm
- net Net-(R14-Pad2): track 37.7 -> 4.86 mm
- net BTN1: track 93.3 -> 61.4 mm
- net BTN3: track 99.8 -> 68.8 mm
- net Net-(J1-Pad7): track 2.23 -> 29.2 mm
- net DISDIGI3: track 14.9 -> 40.3 mm
- net DISDATA: track 29.5 -> 54.0 mm
- net Net-(R16-Pad2): track 0.00 -> 23.9 mm
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Other:
- board size 54.3 x 59.4 mm -> 96.5 x 68.6 mm
